File: basic_esp_board.sch (KiCad schematic (older format))
At the start: 20 parts, among them P2 HEADER_1, P3 HEADER_2, P4 HEADER_3, P6 WS2812, Q1 BSS138, Q2 BSS138, SW1 SW_PUSH, U1 ESP-12E, U2 LD1117S33TR, U3 AM2302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

Commit message: Added Lithium Battery Charger with Load Sharing.
Parts:
- added BAT1: BAT, symbol BAT
- added C5, C6: 4u7, symbol C
- added D1: LED, symbol LED
- added R6: 47k, symbol R
- added U5: MCP73831, symbol MCP73831
- R4: value 47K -> 10K
Connections:
- wire segments 80 -> 123
Other:
- moved on the sheet: C3, C4, U2

Commit message: Added PDF plot.
Parts:
- removed BAT1: BAT, symbol BAT
Connections:
- net labels added: BAT
- wire segments 123 -> 96

Commit message: Fixed some of the circuits and merged transistors.
Parts:
- removed Q1, Q2: BSS138, SOT-23, symbol BSS138
- added Q1: BSS138DW, SOT-23, symbol BSS138DW
- added R7: 470, symbol R
- R6: value 47k -> 2k
Connections:
- wire segments 96 -> 126
Other:
- moved on the sheet: C1, C4, P4, R1, R2

Commit message: Initial cut sent for first run.
Parts:
- removed U4: FTDI_BASIC, symbol FTDI_BASIC
- added BT1: BATTERY, Pin_Headers:Pin_Header_Straight_1x02, symbol BATTERY
- added CON1: USB-MICRO-B, Connect:USB_Micro-B, symbol USB-MICRO-B
- added P1: CONN_SERIAL_SF, Pin_Headers:Pin_Header_Straight_1x06, symbol CONN_SERIAL_SF
- C1, C2, C3, C4, C5, C6: footprint (none) -> Capacitors_SMD:C_0805
- D1: footprint (none) -> LEDs:LED-0805
- P2, P3: footprint (none) -> Socket_Strips:Socket_Strip_Straight_1x11
- P4: footprint (none) -> Socket_Strips:Socket_Strip_Straight_1x08
- P6: footprint (none) -> Pin_Headers:Pin_Header_Straight_1x03
- Q1: footprint SOT-23 -> Housings_SOT-23_SOT-143_TSOT-6:SOT-23-6
- R1, R2, R3, R4, R5, R6, R7: footprint (none) -> Resistors_SMD:R_0805
- SW1: footprint (none) -> mage_mega:1107G
- U1: footprint (none) -> ESP8266:ESP-12E
- U2: footprint SOT-223 -> SMD_Packages:SOT-223
- U3: footprint (none) -> Pin_Headers:Pin_Header_Straight_1x04
- U5: footprint (none) -> Housings_SOT-23_SOT-143_TSOT-6:SOT-23-5
Connections:
- net labels removed: BAT
- wire segments 126 -> 114
- no-connect marks 0 -> 6

Commit message: Rejigged the board based on feedback from @projectgus
Parts:
- removed C1: 2u2, Capacitors_SMD:C_0805, symbol C
- removed C2: 0.1u, Capacitors_SMD:C_0805, symbol C
- removed C3: 100nF, Capacitors_SMD:C_0805, symbol C
- removed C4: 10uF, Capacitors_SMD:C_0805, symbol C
- removed Q1: BSS138DW, Housings_SOT-23_SOT-143_TSOT-6:SOT-23-6, symbol BSS138DW
- added C1: 47uF 6.3V, symbol CP
- added R8, R9: 10K, symbol R
- added SW2: RESET, symbol SW_PUSH
- R1: value 470K -> 4.7k; footprint Resistors_SMD:R_0805 -> (none)
- R2: value 100K -> 4.7k; footprint Resistors_SMD:R_0805 -> (none)
- SW1: value SW_PUSH -> PROG; footprint mage_mega:1107G -> (none)
- U2: value LD1117S33TR -> AP2111H-3.3
- U3: value AM2302 -> DHT22
Connections:
- net labels added: +BATT
- wire segments 114 -> 135
- no-connect marks 6 -> 5
Other:
- moved on the sheet: P1

Commit message: Add pullup on GPIO2, change LDO type again, add FT footprint module and Hirose ZX62 USB connector
Parts:
- removed C1: 47uF 6.3V, symbol CP
- removed CON1: USB-MICRO-B, Connect:USB_Micro-B, symbol USB-MICRO-B
- removed U2: AP2111H-3.3, SMD_Packages:SOT-223, symbol LD1117S33TR
- added C1: 100uF 6.3V X5R, Capacitors_SMD:C_1210_HandSoldering, symbol C
- added P5: USB_B, molex_usb:USBMICROB_HIROSE_ZX62_B_5PA, symbol USB_B
- added R10: 10K, Resistors_SMD:R_0805_HandSoldering, symbol R-RESCUE-basic_esp_board
- added U2: TC1262-33VDB, SMD_Packages:SOT-223, symbol LT1129CST-3.3
- C5, C6: footprint Capacitors_SMD:C_0805 -> Capacitors_SMD:C_0805_HandSoldering; symbol C -> C-RESCUE-basic_esp_board
- D1: symbol LED -> LED-RESCUE-basic_esp_board
- R1, R2, R8, R9: footprint (none) -> Resistors_SMD:R_0805_HandSoldering; symbol R -> R-RESCUE-basic_esp_board
- R3, R4, R5, R6, R7: footprint Resistors_SMD:R_0805 -> Resistors_SMD:R_0805_HandSoldering; symbol R -> R-RESCUE-basic_esp_board
- SW1, SW2: footprint (none) -> FT:SW_PUSHBUTTON_PTH
Connections:
- net labels added: ADC, CS0, EN, GPIO10, GPIO12, GPIO13, GPIO14, GPIO15, GPIO16, GPIO2, GPIO4, GPIO5, GPIO9, MISO, MOSI, RXD, SCLK, TXD
- wire segments 135 -> 109
- no-connect marks 5 -> 4
